File: hardware/LogeekRover.kicad_pcb (KiCad board)
At the start: 2 copper layers, 55.9 x 96.5 mm, 59 parts, among them M1 Mounting_Hole, M2 Mounting_Hole, M3 Mounting_Hole, M4 Mounting_Hole, M5 Motor, M6 Motor, M7 Motor, M8 Motor, P1 CONN_01X01, P10 CONN_01X03, P11 CONN_01X03, P12 CONN_01X01, P13 CONN_01X01, P14 CONN_01X03, P15 CONN_01X03, P16 CONN_01X01, P17 CONN_01X01, P18 CONN_01X03, P19 CONN_01X03, P2 CONN_01X03, P20 CONN_01X01, P22 CONN_01X01, P23 CONN_01X03, P24 CONN_01X03, P25 CONN_01X01, P28 CONN_01X01, P29 CONN_01X03, P3 CONN_01X03, P30 CONN_01X02, P31 CONN_01X02, P32 CONN_01X01, P33 CONN_01X03, P34 CONN_01X02, P35 CONN_01X01, P36 CONN_01X03, P39 CONN_01X01, P4 CONN_01X01, P40 CONN_01X03, P41 CONN_01X01, P42 CONN_01X03, P43 CONN_01X01, P44 CONN_01X03, P46 CONN_01X03, P47 CONN_01X02, P48 CONN_01X03, P5 CONN_01X01, P50 CONN_01X03, P52 CONN_01X03, P53 BATT CASE, P54 CONN_01X02, P6 CONN_01X03, P7 CONN_01X03, P8 CONN_01X01, P9 CONN_01X01, U1 L9110S

Commit message: Nightly Backup.
Parts:
- added BT1: Battery, local:Battery_Case_AAAx2, B.Cu at (76.8, 104.1)
- M1, M2, M3, M4: footprint Mounting_Holes:MountingHole_3mm -> local:Mounting_Hole_3mm
- moved P53 95.2 mm to (99.1, 104.1), turned to 270 degrees
- moved P47 2.54 mm to (55.9, 64.8)
- moved P54 2.54 mm to (55.9, 67.3)
- moved P25 1.80 mm to (87.6, 67.3)
- moved P12 1.80 mm to (80.0, 67.3)
- moved P16 1.80 mm to (82.5, 67.3)
- moved P20 1.80 mm to (85.1, 67.3)
- moved P4 1.80 mm to (74.9, 67.3)
- moved P8 1.80 mm to (77.5, 67.3)
- moved P1 1.27 mm to (69.8, 141.0)
- moved P13 1.27 mm to (77.5, 141.0)
- moved P17 1.27 mm to (80.0, 141.0)
- moved P22 1.27 mm to (82.5, 141.0)
- moved P24 1.27 mm to (87.6, 62.2)
- moved P28 1.27 mm to (85.1, 141.0)
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Other:
- outline, holes or cut-outs redrawn

Commit message: Nightly backup.
Parts:
- added C3: 1uF, Capacitors_SMD:C_0603_HandSoldering, F.Cu at (155.7, 123.4)
- added C4: 100nF, Capacitors_SMD:C_0603_HandSoldering, F.Cu at (146.7, 131.4)
- added C5: 1uF, Capacitors_SMD:C_0603_HandSoldering, F.Cu at (156.9, 117.4)
- added C6: 1uF, Capacitors_SMD:C_0603_HandSoldering, F.Cu at (161.2, 117.4)
- added C7: 100nF, Capacitors_SMD:C_0603_HandSoldering, F.Cu at (151.9, 131.4)
- added C8: 100nF, Capacitors_SMD:C_0603_HandSoldering, F.Cu at (165.9, 117.4)
- added D3: Red, LEDs:LED-0603, F.Cu at (165.7, 133.2)
- added D4: Green, LEDs:LED-0603, F.Cu at (166.1, 128.6)
- added D5: Red, LEDs:LED-0603, F.Cu at (170.3, 127.2)
- added D6: Red, LEDs:LED-0603, F.Cu at (178.4, 122.6)
- added D7: Green, LEDs:LED-0603, F.Cu at (169.3, 122.6)
- added D8: Green, LEDs:LED-0603, F.Cu at (161.6, 134.6)
- added M10: Mounting_Hole, local:Mounting_Hole_3mm, F.Cu at (98.7, 78.7)
- added M9: Mounting_Hole, local:Mounting_Hole_3mm, F.Cu at (58.8, 78.7)
- added P21: Logeek_Socket, local:Logeek_Socket_SMD, F.Cu at (52.1, 69.8)
- added R1: 1k, Resistors_SMD:R_0603_HandSoldering, F.Cu at (160.1, 123.4)
- added R2: 240, Resistors_SMD:R_0603_HandSoldering, F.Cu at (164.6, 123.4)
- added R3: 1k, Resistors_SMD:R_0603_HandSoldering, F.Cu at (170.8, 117.4)
- added R4: 240, Resistors_SMD:R_0603_HandSoldering, F.Cu at (156.8, 129.4)
- added R5: 1k, Resistors_SMD:R_0603_HandSoldering, F.Cu at (161.4, 129.4)
- added R6: 1k, Resistors_SMD:R_0603_HandSoldering, F.Cu at (156.8, 135.4)
- added R7: 240, Resistors_SMD:R_0603_HandSoldering, F.Cu at (175.4, 117.4)
- added R8: 240, Resistors_SMD:R_0603_HandSoldering, F.Cu at (152.5, 117.4)
- added U2: L9110S, SMD_Packages:SOIC-8-N, F.Cu at (72.4, 97.8)
- added U3: L9110S, SMD_Packages:SOIC-8-N, F.Cu at (72.4, 110.5)
- added U4: L9110S, SMD_Packages:SOIC-8-N, F.Cu at (85.1, 110.5)
- moved U1 103.3 mm to (85.1, 97.8), turned to 90 degrees
- moved C1 86.0 mm to (151.4, 125.4)
- moved P34 78.7 mm to (101.6, 64.8)
- moved C2 74.1 mm to (146.7, 125.4)
- moved D1 64.3 mm to (173.7, 127.2)
- moved P39 48.3 mm to (101.6, 141.0)
- moved P41 48.3 mm to (104.1, 141.0)
- moved D2 40.0 mm to (174.2, 122.6)
- moved P53 11.1 mm to (101.6, 93.3)
- moved P35 2.54 mm to (55.9, 141.0)
Connections:
- M6 pad 1: Net-(M6-Pad1) -> /M2R
- M6 pad 2: Net-(M6-Pad2) -> /M2F
- M7 pad 1: Net-(M7-Pad1) -> /M3R
- M7 pad 2: Net-(M7-Pad2) -> /M3F
- M8 pad 1: Net-(M8-Pad1) -> /M4F
- M8 pad 2: Net-(M8-Pad2) -> /M4R
Other:
- outline, holes or cut-outs redrawn

Commit message: Nightly backup.
Parts:
- removed P53: BATT CASE, Connect:PINHEAD1-2
- added SW1: SWITCH_INV, local:SS-12D07, B.Cu at (78.7, 119.4)
- moved U1 2.54 mm to (85.1, 95.2)
- moved U2 2.54 mm to (72.4, 95.2)
- moved U3 2.54 mm to (72.4, 113.0)
- moved U4 2.54 mm to (85.1, 113.0)
- moved BT1 1.91 mm to (78.7, 104.1)
Connections:
- BT1 pad 1: VCC -> Net-(BT1-Pad1)
- C1 pad 2: VCC -> +BATT
- C3 pad 2: VCC -> +BATT
- C5 pad 2: VCC -> +BATT
- C6 pad 2: VCC -> +BATT
- P21 pad A7: VCC -> /VCC
- P34 pad 1: /VIN -> /VCC
- U1 pad 2: VCC -> +BATT
- U1 pad 3: VCC -> +BATT
- U2 pad 2: VCC -> +BATT
- U2 pad 3: VCC -> +BATT
- U3 pad 2: VCC -> +BATT
- U3 pad 3: VCC -> +BATT
- U4 pad 2: VCC -> +BATT
- U4 pad 3: VCC -> +BATT
Other:
- outline, holes or cut-outs redrawn

Commit message: Daily backup.
Parts:
- removed P11, P14, P15, P18, P19, P23, P24, P29, P33, P36, P40, P42, P44, P46, P48, P50, P52: CONN_01X03, Socket_Strips:Socket_Strip_Straight_1x03
- removed P12, P13, P16, P17, P20, P22, P25, P28, P32, P35, P39, P41, P43: CONN_01X01, Socket_Strips:Socket_Strip_Straight_1x01
- removed P30, P31, P34, P47, P54: CONN_01X02, Socket_Strips:Socket_Strip_Straight_1x02
- added R10: 1k, Resistors_SMD:R_0603_HandSoldering, F.Cu at (110.1, 184.0)
- added R11: 1k, Resistors_SMD:R_0603_HandSoldering, F.Cu at (118.6, 178.0)
- added R12: 1k, Resistors_SMD:R_0603_HandSoldering, F.Cu at (114.6, 184.0)
- added R9: 1k, Resistors_SMD:R_0603_HandSoldering, F.Cu at (114.0, 178.0)
- P1, P4, P8: value CONN_01X01 -> CONN_01X06; footprint Socket_Strips:Socket_Strip_Straight_1x01 -> Socket_Strips:Socket_Strip_Straight_1x06
- P10: value CONN_01X03 -> CONN_01X08; footprint Socket_Strips:Socket_Strip_Straight_1x03 -> Socket_Strips:Socket_Strip_Straight_1x08
- P2, P3: value CONN_01X03 -> CONN_01X16; footprint Socket_Strips:Socket_Strip_Straight_1x03 -> Socket_Strips:Socket_Strip_Straight_1x16
- P5: value CONN_01X01 -> CONN_01X16; footprint Socket_Strips:Socket_Strip_Straight_1x01 -> Socket_Strips:Socket_Strip_Straight_1x16
- P6: value CONN_01X03 -> CONN_01X06; footprint Socket_Strips:Socket_Strip_Straight_1x03 -> Socket_Strips:Socket_Strip_Straight_1x06
- P7: value CONN_01X03 -> CONN_01X04; footprint Socket_Strips:Socket_Strip_Straight_1x03 -> Socket_Strips:Socket_Strip_Straight_1x04
- P9: value CONN_01X01 -> CONN_01X04; footprint Socket_Strips:Socket_Strip_Straight_1x01 -> Socket_Strips:Socket_Strip_Straight_1x04
- moved D5 129.7 mm to (55.9, 66.0)
- moved D7 129.1 mm to (53.3, 66.0)
- moved D6 126.6 mm to (53.3, 142.2)
- moved D8 105.9 mm to (55.9, 142.2)
- moved R7 96.5 mm to (105.5, 184.0)
- moved D1 94.5 mm to (101.6, 66.0)
- moved P6 92.3 mm to (74.9, 59.7), turned to 0 degrees
- moved D2 90.1 mm to (104.1, 66.0)
- moved C6 89.5 mm to (95.3, 178.0)
- moved R3 89.5 mm to (104.9, 178.0)
- moved R1 87.9 mm to (96.4, 184.0)
- moved P3 87.7 mm to (59.7, 148.6), turned to 0 degrees
- moved P9 85.2 mm to (90.2, 57.1)
- moved C8 81.6 mm to (105.3, 172.0)
- moved C1 80.1 mm to (91.0, 178.0)
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Connections:
- P1 pad 1: /B0 -> /RXD
- P10 pad 1: GND -> /B0
- P10 pad 2: /VIO -> /B1
- P10 pad 3: /C2 -> /B2
- P2 pad 2: /VIO -> GND
- P2 pad 3: /C0 -> GND
- P21 pad A7: /VCC -> +BATT
- P21 pad B2: GNDA -> GND
- P21 pad D3: /M3A -> /M4A
- P21 pad D5: /M3B -> /M4B
- P21 pad D8: /M4A -> /M3A
- P21 pad D9: /M4B -> /M3B
- P3 pad 1: /M3S -> /VIO
- P3 pad 3: GND -> /VIO
- P4 pad 1: /M3B -> /A4
- P5 pad 1: /B1 -> /C0
- P6 pad 1: GND -> /VIO
- P6 pad 3: /C1 -> /VIO
- P7 pad 1: /M4S -> /RST
- P7 pad 2: /VIO -> /3.3V
- P7 pad 3: GND -> /5V
- P8 pad 1: /M3A -> GND
- P9 pad 1: /B2 -> GND
