File: hardware/LogeekRover.sch (KiCad schematic (older format))
At the start: 17 parts

Commit message: Daily backup.
Parts:
- removed P?: XH2.54 2PIN, symbol CONN_01X02
- removed P? (x2): CONN_01X10, symbol CONN_01X10
- removed P? (x4): CONN_01X08, symbol CONN_01X08
- removed P? (x2): CONN_01X06, symbol CONN_01X06
- added M1, M2, M3, M4: Mounting_Hole, Mounting_Holes:MountingHole_3mm, symbol Mounting_Hole
- added M5, M6, M7, M8: Motor, local:N20_Mount_Rack, symbol Motor
- added P1, P12, P13, P16, P17, P20, P22, P25, P28, P32, P35, P39, P4, P41, P43, P5, P8, P9: CONN_01X01, Socket_Strips:Socket_Strip_Straight_1x01, symbol CONN_01X01
- added P10, P11, P14, P15, P18, P19, P2, P23, P24, P29, P3, P33, P36, P40, P42, P44, P46, P48, P50, P52, P6, P7: CONN_01X03, Socket_Strips:Socket_Strip_Straight_1x03, symbol CONN_01X03
- added P26: CONN_02X10, symbol CONN_02X10
- added P27, P37: CONN_02X08, symbol CONN_02X08
- added P30, P31, P34, P47, P54: CONN_01X02, Socket_Strips:Socket_Strip_Straight_1x02, symbol CONN_01X02
- added P38: CONN_02X06, symbol CONN_02X06
- P53: renamed from P?; footprint (none) -> Connect:PINHEAD1-2
- gave numbers to parts that had none: 7
Connections:
- net labels added: CLK, RST, VIN, VIO
- net labels removed: EXTCLK, IOREF, RESETn
- wire segments 105 -> 188
Other:
- moved on the sheet: P53

Commit message: Nightly Backup.
Parts:
- added BT1: Battery, local:Battery_Case_AAAx2, symbol Battery
- M1, M2, M3, M4: footprint Mounting_Holes:MountingHole_3mm -> local:Mounting_Hole_3mm
Connections:
- wire segments 188 -> 192
Other:
- moved on the sheet: P53
Changed lines of the file:
@@
 	2500 1000 4200 1000
 $Comp
-L VCC #PWR01
+L VCC #PWR2
 U 1 1 56A5EDCA
 P 2400 900
-F 0 "#PWR01" H 2400 750 50  0001 C CNN
+F 0 "#PWR2" H 2400 750 50  0001 C CNN
 F 1 "VCC" H 2400 1050 50  0000 C CNN
 F 2 "" H 2400 900 60  0000 C CNN
@@
 	3750 2000 3750 1900
 $Comp
-L GND #PWR02
+L GND #PWR4
 U 1 1 56A5FD75
 P 3750 2350
-F 0 "#PWR02" H 3750 2100 50  0001 C CNN
+F 0 "#PWR4" H 3750 2100 50  0001 C CNN
 F 1 "GND" H 3750 2200 50  0000 C CNN
 F 2 "" H 3750 2350 60  0000 C CNN
@@
 L CONN_01X02 P53
 U 1 1 56A607A9
-P 12550 8900
-F 0 "P53" H 12550 9050 50  0000 C CNN
-F 1 "BATT CASE" V 12650 8900 50  0000 C CNN
-F 2 "Connect:PINHEAD1-2" H 12550 8900 60  0001 C CNN
-F 3 "" H 12550 8900 60  0000 C CNN
-	1    12550 8900
-	1    0    0    -1
-$EndComp
-$Comp
-L VCC #PWR03
+P 13000 8900
+F 0 "P53" H 13000 9050 50  0000 C CNN
+F 1 "BATT CASE" V 13100 8900 50  0000 C CNN
+F 2 "Connect:PINHEAD1-2" H 13000 8900 60  0001 C CNN
+F 3 "" H 13000 8900 60  0000 C CNN
+	1    13000 8900
+	1    0    0    -1
+$EndComp
+$Comp
+L VCC #PWR8
 U 1 1 56A6091B
-P 12200 8800
-F 0 "#PWR03" H 12200 8650 50  0001 C CNN
-F 1 "VCC" H 12200 8950 50  0000 C CNN
-F 2 "" H 12200 8800 60  0000 C CNN
-F 3 "" H 12200 8800 60  0000 C CNN
-	1    12200 8800
-	1    0    0    -1
-$EndComp
-$Comp
-L GND #PWR04
+P 12200 8600
+F 0 "#PWR8" H 12200 8450 50  0001 C CNN
+F 1 "VCC" H 12200 8750 50  0000 C CNN
+F 2 "" H 12200 8600 60  0000 C CNN
+F 3 "" H 12200 8600 60  0000 C CNN
+	1    12200 8600
+	1    0    0    -1
+$EndComp
+$Comp
+L GND #PWR9
 U 1 1 56A60944
-P 12200 9000
-F 0 "#PWR04" H 12200 8750 50  0001 C CNN
-F 1 "GND" H 12200 8850 50  0000 C CNN
-F 2 "" H 12200 9000 60  0000 C CNN
-F 3 "" H 12200 9000 60  0000 C CNN
-	1    12200 9000
-	1    0    0    -1
-$EndComp
-Wire Wire Line
-	12350 8850 12200 8850
-Wire Wire Line
-	12200 8850 12200 8800
-Wire Wire Line
-	12350 8950 12200 8950
-Wire Wire Line
-	12200 8950 12200 9000
-$Comp
-L GND #PWR05
+P 12200 9200
+F 0 "#PWR9" H 12200 8950 50  0001 C CNN
+F 1 "GND" H 12200 9050 50  0000 C CNN
+F 2 "" H 12200 9200 60  0000 C CNN
+F 3 "" H 12200 9200 60  0000 C CNN
+	1    12200 9200
+	1    0    0    -1
+$EndComp
+$Comp
+L GND #PWR1
 U 1 1 56A60B6D
 P 1200 1900
-F 0 "#PWR05" H 1200 1650 50  0001 C CNN
+F 0 "#PWR1" H 1200 1650 50  0001 C CNN
 F 1 "GND" H 1200 1750 50  0000 C CNN
 F 2 "" H 1200 1900 60  0000 C CNN
@@
 5V
 $Comp
-L GND #PWR06
+L GND #PWR7
 U 1 1 56A6424E
 P 7100 8450
-F 0 "#PWR06" H 7100 8200 50  0001 C CNN
+F 0 "#PWR7" H 7100 8200 50  0001 C CNN
 F 1 "GND" H 7100 8300 50  0000 C CNN
 F 2 "" H 7100 8450 60  0000 C CNN
@@
 AREF
 $Comp
-L GND #PWR07
+L GND #PWR3
 U 1 1 56A6454B
 P 3600 7850
-F 0 "#PWR07" H 3600 7600 50  0001 C CNN
+F 0 "#PWR3" H 3600 7600 50  0001 C CNN
 F 1 "GND" H 3600 7700 50  0000 C CNN
 F 2 "" H 3600 7850 60  0000 C CNN
@@
 CLK
 $Comp
-L GND #PWR08
+L GND #PWR5
 U 1 1 56A6516D
 P 5350 7550
-F 0 "#PWR08" H 5350 7300 50  0001 C CNN
+F 0 "#PWR5" H 5350 7300 50  0001 C CNN
 F 1 "GND" H 5350 7400 50  0000 C CNN
 F 2 "" H 5350 7550 60  0000 C CNN
@@
 A5
 $Comp
-L GNDA #PWR09
+L GNDA #PWR6
 U 1 1 56A65651
 P 5500 9300
-F 0 "#PWR09" H 5500 9050 50  0001 C CNN
+F 0 "#PWR6" H 5500 9050 50  0001 C CNN
 F 1 "GNDA" H 5500 9150 50  0000 C CNN
 F 2 "" H 5500 9300 60  0000 C CNN
@@
 F 0 "M1" H 10650 1850 60  0000 C CNN
 F 1 "Mounting_Hole" H 10700 1550 60  0001 C CNN
-F 2 "Mounting_Holes:MountingHole_3mm" H 10700 1700 60  0001 C CNN
+F 2 "local:Mounting_Hole_3mm" H 10700 1700 60  0001 C CNN
 F 3 "" H 10700 1700 60  0000 C CNN
 	1    10700 1700
@@
 F 0 "M2" H 10950 1850 60  0000 C CNN
 F 1 "Mounting_Hole" H 11000 1550 60  0001 C CNN
-F 2 "Mounting_Holes:MountingHole_3mm" H 11000 1700 60  0001 C CNN
+F 2 "local:Mounting_Hole_3mm" H 11000 1700 60  0001 C CNN
 F 3 "" H 11000 1700 60  0000 C CNN
 	1    11000 1700
@@
 F 0 "M3" H 11250 1850 60  0000 C CNN
 F 1 "Mounting_Hole" H 11300 1550 60  0001 C CNN
-F 2 "Mounting_Holes:MountingHole_3mm" H 11300 1700 60  0001 C CNN
+F 2 "local:Mounting_Hole_3mm" H 11300 1700 60  0001 C CNN
 F 3 "" H 11300 1700 60  0000 C CNN
 	1    11300 1700
@@
 F 0 "M4" H 11550 1850 60  0000 C CNN
 F 1 "Mounting_Hole" H 11600 1550 60  0001 C CNN
-F 2 "Mounting_Holes:MountingHole_3mm" H 11600 1700 60  0001 C CNN
+F 2 "local:Mounting_Hole_3mm" H 11600 1700 60  0001 C CNN
 F 3 "" H 11600 1700 60  0000 C CNN
 	1    11600 1700
@@
 Wire Wire Line
 	3700 1600 4200 1600
+$Comp
+L Battery BT1
+U 1 1 56A8C54E
+P 12200 8900
+F 0 "BT1" H 12300 8950 50  0000 L CNN
+F 1 "Battery" H 12300 8850 50  0000 L CNN
+F 2 "local:Battery_Case_AAAx2" V 12200 8940 60  0001 C CNN
+F 3 "" V 12200 8940 60  0000 C CNN
+	1    12200 8900
+	1    0    0    -1
+$EndComp
+Wire Wire Line
+	12200 8600 12200 8750
+Wire Wire Line
+	12200 9050 12200 9200
+Wire Wire Line
+	12200 8650 12650 8650
+Wire Wire Line
+	12650 8650 12650 8850
+Wire Wire Line
+	12650 8850 12800 8850
+Connection ~ 12200 8650
+Wire Wire Line
+	12800 8950 12650 8950
+Wire Wire Line
+	12650 8950 12650 9150
+Wire Wire Line
+	12650 9150 12200 9150
+Connection ~ 12200 9150
 $EndSCHEMATC

Commit message: Nightly backup.
Parts:
- removed P26: CONN_02X10, symbol CONN_02X10
- removed P27, P37: CONN_02X08, symbol CONN_02X08
- removed P38: CONN_02X06, symbol CONN_02X06
- added C3, C5, C6: 1uF, Capacitors_SMD:C_0603_HandSoldering, symbol C
- added C4, C7, C8: 100nF, Capacitors_SMD:C_0603_HandSoldering, symbol C
- added D3, D5, D6: Red, LEDs:LED-0603, symbol LED
- added D4, D7, D8: Green, LEDs:LED-0603, symbol LED
- added M10, M9: Mounting_Hole, local:Mounting_Hole_3mm, symbol Mounting_Hole
- added P21: Logeek_Socket, local:Logeek_Socket_SMD, symbol Logeek_Socket
- added R3, R5, R6: 1k, Resistors_SMD:R_0603_HandSoldering, symbol R
- added R4, R7, R8: 240, Resistors_SMD:R_0603_HandSoldering, symbol R
- added U2, U3, U4: L9110S, SMD_Packages:SOIC-8-N, symbol L9110
- R1, R2: footprint (none) -> Resistors_SMD:R_0603_HandSoldering
Connections:
- net labels added: M2F, M2R, M3F, M3R, M4F, M4R
- wire segments 192 -> 270
Other:
- moved on the sheet: M1, M2, M3, M4, M6, M7, M8, P11, P12, P15, P16, P19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

Commit message: Nightly backup.
Parts:
- removed P53: BATT CASE, Connect:PINHEAD1-2, symbol CONN_01X02
- added SW1: SWITCH_INV, local:SS-12D07, symbol SWITCH_INV
Connections:
- net labels added: +BATT
- net labels removed: VIN
- wire segments 270 -> 268
Other:
- moved on the sheet: BT1, P34, P54
Changed lines of the file:
@@
 Wire Wire Line
 	2500 1000 4200 1000
-$Comp
-L VCC #PWR01
-U 1 1 56A5EDCA
-P 2400 900
-F 0 "#PWR01" H 2400 750 50  0001 C CNN
-F 1 "VCC" H 2400 1050 50  0000 C CNN
-F 2 "" H 2400 900 60  0000 C CNN
-F 3 "" H 2400 900 60  0000 C CNN
-	1    2400 900
-	1    0    0    -1
-$EndComp
 Wire Wire Line
 	2400 1600 2300 1600
@@
 	3750 2000 3750 1900
 $Comp
-L GND #PWR02
+L GND #PWR5
 U 1 1 56A5FD75
 P 3750 2350
-F 0 "#PWR02" H 3750 2100 50  0001 C CNN
+F 0 "#PWR5" H 3750 2100 50  0001 C CNN
 F 1 "GND" H 3750 2200 50  0000 C CNN
 F 2 "" H 3750 2350 60  0000 C CNN
@@
 	3750 2300 3750 2350
 $Comp
-L CONN_01X02 P53
-U 1 1 56A607A9
-P 13000 8900
-F 0 "P53" H 13000 9050 50  0000 C CNN
-F 1 "BATT CASE" V 13100 8900 50  0000 C CNN
-F 2 "Connect:PINHEAD1-2" H 13000 8900 60  0001 C CNN
-F 3 "" H 13000 8900 60  0000 C CNN
-	1    13000 8900
-	1    0    0    -1
-$EndComp
-$Comp
-L VCC #PWR03
+L +BATT #PWR18
 U 1 1 56A6091B
-P 12200 8600
-F 0 "#PWR03" H 12200 8450 50  0001 C CNN
-F 1 "VCC" H 12200 8750 50  0000 C CNN
-F 2 "" H 12200 8600 60  0000 C CNN
-F 3 "" H 12200 8600 60  0000 C CNN
-	1    12200 8600
-	1    0    0    -1
-$EndComp
-$Comp
-L GND #PWR04
-U 1 1 56A60944
-P 12200 9200
-F 0 "#PWR04" H 12200 8950 50  0001 C CNN
-F 1 "GND" H 12200 9050 50  0000 C CNN
-F 2 "" H 12200 9200 60  0000 C CNN
-F 3 "" H 12200 9200 60  0000 C CNN
-	1    12200 9200
-	1    0    0    -1
-$EndComp
-$Comp
-L GND #PWR05
+P 14200 8650
+F 0 "#PWR18" H 14200 8500 50  0001 C CNN
+F 1 "+BATT" H 14200 8800 50  0000 C CNN
+F 2 "" H 14200 8650 60  0000 C CNN
+F 3 "" H 14200 8650 60  0000 C CNN
+	1    14200 8650
+	1    0    0    -1
+$EndComp
+$Comp
+L GND #PWR1
 U 1 1 56A60B6D
 P 1200 1900
-F 0 "#PWR05" H 1200 1650 50  0001 C CNN
+F 0 "#PWR1" H 1200 1650 50  0001 C CNN
 F 1 "GND" H 1200 1750 50  0000 C CNN
 F 2 "" H 1200 1900 60  0000 C CNN
@@
 5V
 $Comp
-L GND #PWR06
+L GND #PWR17
 U 1 1 56A6424E
 P 14100 5800
-F 0 "#PWR06" H 14100 5550 50  0001 C CNN
+F 0 "#PWR17" H 14100 5550 50  0001 C CNN
 F 1 "GND" H 14100 5650 50  0000 C CNN
 F 2 "" H 14100 5800 60  0000 C CNN
@@
 AREF
 $Comp
-L GND #PWR07
+L GND #PWR13
 U 1 1 56A6454B
 P 11100 5150
-F 0 "#PWR07" H 11100 4900 50  0001 C CNN
+F 0 "#PWR13" H 11100 4900 50  0001 C CNN
 F 1 "GND" H 11100 5000 50  0000 C CNN
 F 2 "" H 11100 5150 60  0000 C CNN
@@
 CLK
 $Comp
-L GND #PWR08
+L GND #PWR14
 U 1 1 56A6516D
 P 12650 4850
-F 0 "#PWR08" H 12650 4600 50  0001 C CNN
+F 0 "#PWR14" H 12650 4600 50  0001 C CNN
 F 1 "GND" H 12650 4700 50  0000 C CNN
 F 2 "" H 12650 4850 60  0000 C CNN
@@
 A5
 $Comp
-L GNDA #PWR09
+L GNDA #PWR15
 U 1 1 56A65651
 P 13050 6500
-F 0 "#PWR09" H 13050 6250 50  0001 C CNN
+F 0 "#PWR15" H 13050 6250 50  0001 C CNN
 F 1 "GNDA" H 13050 6350 50  0000 C CNN
 F 2 "" H 13050 6500 60  0000 C CNN
@@
 GND
 Wire Wire Line
-	8950 9450 8750 9450
-Wire Wire Line
-	8950 9550 8750 9550
-Text Label 8750 9550 0    60   ~ 0
-VIN
-Text Label 8750 9450 0    60   ~ 0
+	7250 8900 7050 8900
+Wire Wire Line
+	7250 9000 7050 9000
+Text Label 7050 9000 0    60   ~ 0
+VCC
+Text Label 7050 8900 0    60   ~ 0
 GND
 $Comp
@@
 L CONN_01X02 P34
 U 1 1 56A9D286
-P 8550 9500
-F 0 "P34" H 8550 9650 50  0000 C CNN
-F 1 "CONN_01X02" V 8650 9500 50  0001 C CNN
-F 2 "Socket_Strips:Socket_Strip_Straight_1x02" H 8550 9500 60  0001 C CNN
-F 3 "" H 8550 9500 60  0000 C CNN
-	1    8550 9500
+P 6850 8950
+F 0 "P34" H 6850 9100 50  0000 C CNN
+F 1 "CONN_01X02" V 6950 8950 50  0001 C CNN
+F 2 "Socket_Strips:Socket_Strip_Straight_1x02" H 6850 8950 60  0001 C CNN
+F 3 "" H 6850 8950 60  0000 C CNN
+	1    6850 8950
 	-1   0    0    1
 $EndComp
@@
 L CONN_01X02 P54
 U 1 1 56AA3EC9
-P 6750 8450
-F 0 "P54" H 6750 8600 50  0000 C CNN
-F 1 "CONN_01X02" V 6850 8450 50  0001 C CNN
-F 2 "Socket_Strips:Socket_Strip_Straight_1x02" H 6750 8450 60  0001 C CNN
-F 3 "" H 6750 8450 60  0000 C CNN
-	1    6750 8450
-	-1   0    0    1
-$EndComp
-Wire Wire Line
-	7150 8400 6950 8400
-Wire Wire Line
-	7150 8500 6950 8500
-Text Label 6950 8500 0    60   ~ 0
+P 6300 8950
+F 0 "P54" H 6300 9100 50  0000 C CNN
+F 1 "CONN_01X02" V 6400 8950 50  0001 C CNN
+F 2 "Socket_Strips:Socket_Strip_Straight_1x02" H 6300 8950 60  0001 C CNN
+F 3 "" H 6300 8950 60  0000 C CNN
+	1    6300 8950
+	-1   0    0    1
+$EndComp
+Wire Wire Line
+	6700 8900 6500 8900
+Wire Wire Line
+	6700 9000 6500 9000
+Text Label 6500 9000 0    60   ~ 0
 5V
 $Comp
@@
 Text Label 5950 9000 0    60   ~ 0
 3.3V
-Text Label 6950 8400 0    60   ~ 0
+Text Label 6500 8900 0    60   ~ 0
 GND
 Text Label 5950 8900 0    60   ~ 0
@@
 L Battery BT1
 U 1 1 56A8C54E
-P 12200 8900
-F 0 "BT1" H 12300 8950 50  0000 L CNN
-F 1 "Battery" H 12300 8850 50  0000 L CNN
-F 2 "local:Battery_Case_AAAx2" V 12200 8940 60  0001 C CNN
-F 3 "" V 12200 8940 60  0000 C CNN
-	1    12200 8900
-	1    0    0    -1
-$EndComp
-Wire Wire Line
-	12200 8600 12200 8750
-Wire Wire Line
-	12200 9050 12200 9200
-Wire Wire Line
-	12200 8650 12650 8650
-Wire Wire Line
-	12650 8650 12650 8850
-Wire Wire Line
-	12650 8850 12800 8850
-Connection ~ 12200 8650
-Wire Wire Line
-	12800 8950 12650 8950
-Wire Wire Line
-	12650 8950 12650 9150
-Wire Wire Line
-	12650 9150 12200 9150
-Connection ~ 12200 9150
+P 12750 8900
+F 0 "BT1" H 12850 8950 50  0000 L CNN
+F 1 "Battery" H 12850 8850 50  0000 L CNN
+F 2 "local:Battery_Case_AAAx2" V 12750 8940 60  0001 C CNN
+F 3 "" V 12750 8940 60  0000 C CNN
+	1    12750 8900
+	1    0    0    -1
+$EndComp
+Wire Wire Line
+	12750 8650 13200 8650
 $Comp
 L Logeek_Socket P21
@@
 Wire Wire Line
 	2500 2750 4200 2750
-$Comp
-L VCC #PWR010
-U 1 1 56B03370
-P 2400 2650
-F 0 "#PWR010" H 2400 2500 50  0001 C CNN
-F 1 "VCC" H 2400 2800 50  0000 C CNN
-F 2 "" H 2400 2650 60  0000 C CNN
-F 3 "" H 2400 2650 60  0000 C CNN
-	1    2400 2650
-	1    0    0    -1
-$EndComp
 Wire Wire Line
 	2400 3350 2300 3350
@@
 	3750 3750 3750 3650
 $Comp
-L GND #PWR011
+L GND #PWR6
 U 1 1 56B03393
 P 3750 4100
-F 0 "#PWR011" H 3750 3850 50  0001 C CNN
+F 0 "#PWR6" H 3750 3850 50  0001 C CNN
 F 1 "GND" H 3750 3950 50  0000 C CNN
 F 2 "" H 3750 4100 60  0000 C CNN
@@
 	3750 4050 3750 4100
 $Comp
-L GND #PWR012
+L GND #PWR2
 U 1 1 56B033A6
 P 1200 3650
-F 0 "#PWR012" H 1200 3400 50  0001 C CNN
+F 0 "#PWR2" H 1200 3400 50  0001 C CNN
 F 1 "GND" H 1200 3500 50  0000 C CNN
 F 2 "" H 1200 3650 60  0000 C CNN
@@
 Wire Wire Line
 	6350 1000 8050 1000
-$Comp
-L VCC #PWR013
-U 1 1 56B03BD2
-P 6250 900
-F 0 "#PWR013" H 6250 750 50  0001 C CNN
-F 1 "VCC" H 6250 1050 50  0000 C CNN
-F 2 "" H 6250 900 60  0000 C CNN
-F 3 "" H 6250 900 60  0000 C CNN
-	1    6250 900
-	1    0    0    -1
-$EndComp
 Wire Wire Line
 	6250 1600 6150 1600
@@
 	7600 2000 7600 1900
 $Comp
-L GND #PWR014
+L GND #PWR11
 U 1 1 56B03BF5
 P 7600 2350
-F 0 "#PWR014" H 7600 2100 50  0001 C CNN
+F 0 "#PWR11" H 7600 2100 50  0001 C CNN
 F 1 "GND" H 7600 2200 50  0000 C CNN
 F 2 "" H 7600 2350 60  0000 C CNN
@@
 	7600 2300 7600 2350
 $Comp
-L GND #PWR015
+L GND #PWR7
 U 1 1 56B03C08
 P 5050 1900
-F 0 "#PWR015" H 5050 1650 50  0001 C CNN
+F 0 "#PWR7" H 5050 1650 50  0001 C CNN
 F 1 "GND" H 5050 1750 50  0000 C CNN
 F 2 "" H 5050 1900 60  0000 C CNN
@@
 Wire Wire Line
 	6350 2700 8050 2700
-$Comp
-L VCC #PWR016
-U 1 1 56B03F37
-P 6250 2600
-F 0 "#PWR016" H 6250 2450 50  0001 C CNN
-F 1 "VCC" H 6250 2750 50  0000 C CNN
-F 2 "" H 6250 2600 60  0000 C CNN
-F 3 "" H 6250 2600 60  0000 C CNN
-	1    6250 2600
-	1    0    0    -1
-$EndComp
 Wire Wire Line
 	6250 3300 6150 3300
@@
 	7600 3700 7600 3600
 $Comp
-L GND #PWR017
+L GND #PWR12
 U 1 1 56B03F5A
 P 7600 4050
-F 0 "#PWR017" H 7600 3800 50  0001 C CNN
+F 0 "#PWR12" H 7600 3800 50  0001 C CNN
 F 1 "GND" H 7600 3900 50  0000 C CNN
 F 2 "" H 7600 4050 60  0000 C CNN
@@
 	7600 4000 7600 4050
 $Comp
-L GND #PWR018
+L GND #PWR8
 U 1 1 56B03F6D
 P 5050 3600
-F 0 "#PWR018" H 5050 3350 50  0001 C CNN
+F 0 "#PWR8" H 5050 3350 50  0001 C CNN
 F 1 "GND" H 5050 3450 50  0000 C CNN
 F 2 "" H 5050 3600 60  0000 C CNN
@@
 Wire Wire Line
 	7550 3300 8050 3300
+$Comp
+L SWITCH_INV SW1
+U 1 1 56B0D354
+P 13700 8750
+F 0 "SW1" H 13500 8900 50  0000 C CNN
+F 1 "SWITCH_INV" H 13550 8600 50  0000 C CNN
+F 2 "local:SS-12D07" H 13700 8750 60  0001 C CNN
+F 3 "" H 13700 8750 60  0000 C CNN
+	1    13700 8750
+	-1   0    0    1
+$EndComp
+$Comp
+L GND #PWR16
+U 1 1 56B0DAAF
+P 13200 9150
+F 0 "#PWR16" H 13200 8900 50  0001 C CNN
+F 1 "GND" H 13200 9000 50  0000 C CNN
+F 2 "" H 13200 9150 60  0000 C CNN
+F 3 "" H 13200 9150 60  0000 C CNN
+	1    13200 9150
+	1    0    0    -1
+$EndComp
+Wire Wire Line
+	13200 9150 13200 8850
+Wire Wire Line
+	14200 8750 14200 8650
+Wire Wire Line
+	12750 8650 12750 8750
+Wire Wire Line
+	12750 9050 12750 9100
+Wire Wire Line
+	12750 9100 13200 9100
+Connection ~ 13200 9100
+$Comp
+L +BATT #PWR3
+U 1 1 56B193E6
+P 2400 900
+F 0 "#PWR3" H 2400 750 50  0001 C CNN
+F 1 "+BATT" H 2400 1050 50  0000 C CNN
+F 2 "" H 2400 900 60  0000 C CNN
+F 3 "" H 2400 900 60  0000 C CNN
+	1    2400 900
+	1    0    0    -1
+$EndComp
+$Comp
+L +BATT #PWR9
+U 1 1 56B19BAB
+P 6250 900
+F 0 "#PWR9" H 6250 750 50  0001 C CNN
+F 1 "+BATT" H 6250 1050 50  0000 C CNN
+F 2 "" H 6250 900 60  0000 C CNN
+F 3 "" H 6250 900 60  0000 C CNN
+	1    6250 900
+	1    0    0    -1
+$EndComp
+$Comp
+L +BATT #PWR4
+U 1 1 56B1A06A
+P 2400 2650
+F 0 "#PWR4" H 2400 2500 50  0001 C CNN
+F 1 "+BATT" H 2400 2800 50  0000 C CNN
+F 2 "" H 2400 2650 60  0000 C CNN
+F 3 "" H 2400 2650 60  0000 C CNN
+	1    2400 2650
+	1    0    0    -1
+$EndComp
+$Comp
+L +BATT #PWR10
+U 1 1 56B1A177
+P 6250 2600
+F 0 "#PWR10" H 6250 2450 50  0001 C CNN
+F 1 "+BATT" H 6250 2750 50  0000 C CNN
+F 2 "" H 6250 2600 60  0000 C CNN
+F 3 "" H 6250 2600 60  0000 C CNN
+	1    6250 2600
+	1    0    0    -1
+$EndComp
 $EndSCHEMATC

Commit message: Daily backup.
Parts:
- removed P1, P12, P13, P16, P17, P20, P22, P25, P28, P32, P35, P39, P4, P41, P43, P5, P8, P9: CONN_01X01, Socket_Strips:Socket_Strip_Straight_1x01, symbol CONN_01X01
- removed P10, P11, P14, P15, P18, P19, P2, P23, P24, P29, P3, P33, P36, P40, P42, P44, P46, P48, P50, P52, P6, P7: CONN_01X03, Socket_Strips:Socket_Strip_Straight_1x03, symbol CONN_01X03
- removed P30, P31, P34, P47, P54: CONN_01X02, Socket_Strips:Socket_Strip_Straight_1x02, symbol CONN_01X02
- added P1, P4, P6, P8: CONN_01X06, Socket_Strips:Socket_Strip_Straight_1x06, symbol CONN_01X06
- added P10: CONN_01X08, Socket_Strips:Socket_Strip_Straight_1x08, symbol CONN_01X08
- added P2, P3, P5: CONN_01X16, Socket_Strips:Socket_Strip_Straight_1x16, symbol CONN_01X16
- added P7, P9: CONN_01X04, Socket_Strips:Socket_Strip_Straight_1x04, symbol CONN_01X04
- added R10, R11, R12, R9: 1k, Resistors_SMD:R_0603_HandSoldering, symbol R
Connections:
- net labels removed: GNDA, VCC
- wire segments 268 -> 270
